File: hw/KeyboardPCB/KeyboardPCB.kicad_pcb (KiCad board)
At the start: 2 copper layers, 335 x 100 mm, 173 parts, among them IC1 TPS2113ADRBR, IC2 BGM220PC22HNA2R, J1 USB_B_Micro, J2 Conn_01x07_Pin, J3 Conn_01x06_Pin, J4 Conn_02x05_Odd_Even, J5 BATT_POS, J6 BATT_NEG, K1 KEYSW, K10 KEYSW, K11 KEYSW, K12 KEYSW, K13 KEYSW, K14 KEYSW, K15 KEYSW, K16 KEYSW, K17 KEYSW, K18 KEYSW, K19 KEYSW, K2 KEYSW, K20 KEYSW, K21 KEYSW, K22 KEYSW, K23 KEYSW, K24 KEYSW, K25 KEYSW, K26 KEYSW, K27 KEYSW, K28 KEYSW, K29 KEYSW, K3 KEYSW, K30 KEYSW, K31 KEYSW, K32 KEYSW, K33 KEYSW, K34 KEYSW, K35 KEYSW, K36 KEYSW, K37 KEYSW, K38 KEYSW, K39 KEYSW, K4 KEYSW, K40 KEYSW, K41 KEYSW, K42 KEYSW, K43 KEYSW, K44 KEYSW, K45 KEYSW, K46 KEYSW, K47 KEYSW, K48 KEYSW, K49 KEYSW, K5 KEYSW, K50 KEYSW, K51 KEYSW, K52 KEYSW, K53 KEYSW, K54 KEYSW, K55 KEYSW, K56 KEYSW, K57 KEYSW, K58 KEYSW, K59 KEYSW, K6 KEYSW, K60 KEYSW, K61 KEYSW, K62 KEYSW, K7 KEYSW, K8 KEYSW, K9 KEYSW, SW2 BAT_SWITCH, U1 TM4C123GH6PMI7, U2 TPS73633DBV, U3 Adafruit ST7735R, X2 16MHz

Commit message: Slight tweaks
Parts:
- moved J5 0.68 mm to (688.0, 197.4)
Connections:
- IC2 pad 22: unconnected-(IC2-PC00-Pad22) -> /EM4_WAKEUP
- U1 pad 61: GND -> /EM4_WAKEUP
Routing:
- net GND: track 344.2 -> 282.9 mm, vias 20 -> 18
- net /PTI_DOUT: track 17.8 -> 25.2 mm
- net /PTI_DFRAME: track 16.2 -> 22.6 mm
- net /EM4_WAKEUP: track 0.00 -> 2.54 mm
- net /~{RESET}: track 82.5 -> 83.1 mm
- net /col1: track 383.6 -> 384.1 mm
- net /col9: track 226.5 -> 227.0 mm
- net /col0: track 391.2 -> 391.7 mm
- net /col8: track 218.0 -> 218.5 mm
