File: hw/KeyboardPCB/KeyboardPCB.kicad_pcb (KiCad board)
At the start: 2 copper layers, 105 parts, among them J1 USB_B_Micro, J2 Conn_01x05_Pin, U1 TM4C123GH6PMI7, U2 TPS73633DBV, U3 Adafruit ST7735R

Commit message: Added remaining footprints and aligned keys on layout
Parts:
- removed D20, D25, D35, D40, D45, D63, D70, D9: D, Diode_SMD:D_0603_1608Metric_Pad1.05x0.95mm_HandSolder
- added D71: LED, LED_SMD:LED_0603_1608Metric_Pad1.05x0.95mm_HandSolder, F.Cu at (742.8, 191.2)
- added IC1: TPS2113ADRBR, SwitchingICLibrary:SON65P300X300X100-9N-D, F.Cu at (743.2, 187.6)
- added K1: KEYSW, keebs.pretty-master:Mx_Alps_100, F.Cu at (369.6, 184.4)
- added K10: KEYSW, keebs.pretty-master:Mx_Alps_125, F.Cu at (395.8, 259.6)
- added K11: KEYSW, keebs.pretty-master:Mx_Alps_100, F.Cu at (407.5, 184.4)
- added K12: KEYSW, keebs.pretty-master:Mx_Alps_100, F.Cu at (417.0, 203.2)
- added K13: KEYSW, keebs.pretty-master:Mx_Alps_100, F.Cu at (421.8, 222.0)
- added K14: KEYSW, keebs.pretty-master:Mx_Alps_100, F.Cu at (412.4, 240.8)
- added K15: KEYSW, keebs.pretty-master:Mx_Alps_125, F.Cu at (419.6, 259.6)
- added K16: KEYSW, keebs.pretty-master:Mx_Alps_100, F.Cu at (426.5, 184.4)
- added K17: KEYSW, keebs.pretty-master:Mx_Alps_100, F.Cu at (436.0, 203.2)
- added K18: KEYSW, keebs.pretty-master:Mx_Alps_100, F.Cu at (440.7, 222.0)
- added K19: KEYSW, keebs.pretty-master:Mx_Alps_100, F.Cu at (431.3, 240.8)
- added K2: KEYSW, keebs.pretty-master:Mx_Alps_150, F.Cu at (374.4, 203.2)
- added K21: KEYSW, keebs.pretty-master:Mx_Alps_100, F.Cu at (445.4, 184.4)
- added K22: KEYSW, keebs.pretty-master:Mx_Alps_100, F.Cu at (455.0, 203.2)
- added K23: KEYSW, keebs.pretty-master:Mx_Alps_100, F.Cu at (459.7, 222.0)
- added K24: KEYSW, keebs.pretty-master:Mx_Alps_100, F.Cu at (450.3, 240.8)
- added K26: KEYSW, keebs.pretty-master:Mx_Alps_100, F.Cu at (464.4, 184.4)
- added K27: KEYSW, keebs.pretty-master:Mx_Alps_100, F.Cu at (473.9, 203.2)
- added K28: KEYSW, keebs.pretty-master:Mx_Alps_100, F.Cu at (478.6, 222.0)
- added K29: KEYSW, keebs.pretty-master:Mx_Alps_100, F.Cu at (469.2, 240.8)
- added K3: KEYSW, keebs.pretty-master:Mx_Alps_175, F.Cu at (376.7, 222.0)
- added K30: KEYSW, keebs.pretty-master:Mx_Alps_625, F.Cu at (490.7, 259.6)
- added K31: KEYSW, keebs.pretty-master:Mx_Alps_100, F.Cu at (483.3, 184.4)
- added K32: KEYSW, keebs.pretty-master:Mx_Alps_100, F.Cu at (492.9, 203.2)
- added K33: KEYSW, keebs.pretty-master:Mx_Alps_100, F.Cu at (497.6, 222.0)
- added K34: KEYSW, keebs.pretty-master:Mx_Alps_100, F.Cu at (488.2, 240.8)
- added K36: KEYSW, keebs.pretty-master:Mx_Alps_100, F.Cu at (502.3, 184.4)
- added K37: KEYSW, keebs.pretty-master:Mx_Alps_100, F.Cu at (511.8, 203.2)
- added K38: KEYSW, keebs.pretty-master:Mx_Alps_100, F.Cu at (516.5, 222.0)
- added K39: KEYSW, keebs.pretty-master:Mx_Alps_100, F.Cu at (507.1, 240.8)
- added K4: KEYSW, keebs.pretty-master:Mx_Alps_225, F.Cu at (381.5, 240.8)
- added K41: KEYSW, keebs.pretty-master:Mx_Alps_100, F.Cu at (521.3, 184.4)
- added K42: KEYSW, keebs.pretty-master:Mx_Alps_100, F.Cu at (530.8, 203.2)
- added K43: KEYSW, keebs.pretty-master:Mx_Alps_100, F.Cu at (535.5, 222.0)
- added K44: KEYSW, keebs.pretty-master:Mx_Alps_100, F.Cu at (526.1, 240.8)
- added K46: KEYSW, keebs.pretty-master:Mx_Alps_100, F.Cu at (540.2, 184.4)
- added K47: KEYSW, keebs.pretty-master:Mx_Alps_100, F.Cu at (549.7, 203.2)
- added K48: KEYSW, keebs.pretty-master:Mx_Alps_100, F.Cu at (554.4, 222.0)
- added K49: KEYSW, keebs.pretty-master:Mx_Alps_100, F.Cu at (545.0, 240.8)
- added K5: KEYSW, keebs.pretty-master:Mx_Alps_125, F.Cu at (372.0, 259.6)
- added K50: KEYSW, keebs.pretty-master:Mx_Alps_125, F.Cu at (561.8, 259.6)
- added K51: KEYSW, keebs.pretty-master:Mx_Alps_100, F.Cu at (559.2, 184.4)
- added K52: KEYSW, keebs.pretty-master:Mx_Alps_100, F.Cu at (568.7, 203.2)
- added K53: KEYSW, keebs.pretty-master:Mx_Alps_100, F.Cu at (573.4, 222.0)
- added K54: KEYSW, keebs.pretty-master:Mx_Alps_100, F.Cu at (564.0, 240.8)
- added K55: KEYSW, keebs.pretty-master:Mx_Alps_125, F.Cu at (585.5, 259.6)
- added K56: KEYSW, keebs.pretty-master:Mx_Alps_100, F.Cu at (578.1, 184.4)
- added K57: KEYSW, keebs.pretty-master:Mx_Alps_100, F.Cu at (587.7, 203.2)
- added K58: KEYSW, keebs.pretty-master:Mx_Alps_100, F.Cu at (592.3, 222.0)
- added K59: KEYSW, keebs.pretty-master:Mx_Alps_100, F.Cu at (582.9, 240.8)
- added K6: KEYSW, keebs.pretty-master:Mx_Alps_100, F.Cu at (388.6, 184.4)
- added K60: KEYSW, keebs.pretty-master:Mx_Alps_125, F.Cu at (609.1, 259.6)
- added K61: KEYSW, keebs.pretty-master:Mx_Alps_100, F.Cu at (597.1, 184.4)
- added K62: KEYSW, keebs.pretty-master:Mx_Alps_100, F.Cu at (606.6, 203.2)
- added K64: KEYSW, keebs.pretty-master:Mx_Alps_150, F.Cu at (606.6, 240.8)
- added K65: KEYSW, keebs.pretty-master:Mx_Alps_125, F.Cu at (632.7, 259.6)
- added K66: KEYSW, keebs.pretty-master:Mx_Alps_200, F.Cu at (625.6, 184.4)
- added K67: KEYSW, keebs.pretty-master:Mx_Alps_150, F.Cu at (630.3, 203.2)
- added K68: KEYSW, keebs.pretty-master:Mx_Alps_225, F.Cu at (623.2, 222.0)
- added K69: KEYSW, keebs.pretty-master:Mx_Alps_125, F.Cu at (632.7, 240.8)
- added K7: KEYSW, keebs.pretty-master:Mx_Alps_100, F.Cu at (398.1, 203.2)
- added K8: KEYSW, keebs.pretty-master:Mx_Alps_100, F.Cu at (402.8, 222.0)
- added SW1: SW_Push, Button_Switch_THT:SW_PUSH_6mm, F.Cu at (732.0, 180.9)
- added TP1: USB_DM, TestPoint:TestPoint_Pad_2.5x2.5mm, F.Cu at (718.6, 181.2)
- added TP2: USB_DP, TestPoint:TestPoint_Pad_2.5x2.5mm, F.Cu at (718.6, 185.7)
- added TP3: EN, TestPoint:TestPoint_Pad_2.5x2.5mm, F.Cu at (718.6, 190.3)
- added TP4: VBUS, TestPoint:TestPoint_Pad_2.5x2.5mm, F.Cu at (723.2, 181.2)
- added TP5: 3V3, TestPoint:TestPoint_Pad_2.5x2.5mm, F.Cu at (723.2, 185.7)
- added TP6: GND, TestPoint:TestPoint_Pad_2.5x2.5mm, F.Cu at (723.2, 190.3)
- added TP7: IN1, TestPoint:TestPoint_Pad_2.5x2.5mm, F.Cu at (727.7, 181.2)
- added TP8: VBAT, TestPoint:TestPoint_Pad_2.5x2.5mm, F.Cu at (727.7, 185.7)
- added TP9: Switch_OUT, TestPoint:TestPoint_Pad_2.5x2.5mm, F.Cu at (727.7, 190.3)
- added X2: 16MHz, CrystalLibrary:NX5032GA16000000MHZLNCD1, F.Cu at (745.1, 182.1)
- moved BT1 350.6 mm to (382.1, 28.9)
- moved BT2 350.6 mm to (382.1, 47.2)
- moved BT4 350.6 mm to (382.1, 65.5)
- moved C1 350.6 mm to (416.9, 21.0)
- moved C15 350.6 mm to (425.6, 21.0)
- moved C16 350.6 mm to (425.6, 23.5)
- moved C17 350.6 mm to (425.6, 26.1)
- moved C18 350.6 mm to (425.6, 28.6)
- moved C19 350.6 mm to (425.6, 31.1)
- moved C2 350.6 mm to (416.9, 23.5)
- moved C3 350.6 mm to (416.9, 26.1)
- moved C4 350.6 mm to (416.9, 28.6)
- moved C5 350.6 mm to (416.9, 31.1)
- moved C6 350.6 mm to (416.9, 33.6)
- moved C7 350.6 mm to (416.9, 36.1)
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
Commit message: Placed a few more components under keys
Parts:
- moved J1 263.5 mm to (656.9, 180.8)
- moved D5 170.2 mm to (381.6, 254.2), turned to -90 degrees
- moved D4 164.1 mm to (399.5, 247.5), turned to 180 degrees
- moved D3 149.1 mm to (389.6, 228.9), turned to 180 degrees
- moved D2 133.2 mm to (385.2, 209.5), turned to 180 degrees
- moved D1 118.1 mm to (373.6, 188.4), turned to 180 degrees
- moved D10 44.5 mm to (450.4, 81.0), turned to 180 degrees
- moved D8 41.3 mm to (450.4, 86.2), turned to 180 degrees
- moved D7 40.6 mm to (450.4, 88.8), turned to 180 degrees
- moved D6 40.6 mm to (450.4, 91.4), turned to 180 degrees
- moved D11 39.6 mm to (444.0, 102.0), turned to 180 degrees
- moved D12 36.4 mm to (444.0, 99.4), turned to 180 degrees
- moved D13 33.7 mm to (444.0, 96.8), turned to 180 degrees
- moved D19 33.6 mm to (444.0, 81.3), turned to 180 degrees
- moved D21 33.5 mm to (439.6, 102.0), turned to 180 degrees
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
Commit message: Made outline and placed all components in position. Just need to route :)
Parts:
- removed TP3: EN, TestPoint:TestPoint_Pad_2.5x2.5mm
- removed TP4: VBUS, TestPoint:TestPoint_Pad_2.5x2.5mm
- added IC2: BGM220PC22HNA2R, BluetoothModuleLibrary:BGM220PC22HNA2R, F.Cu at (657.1, 200.7)
- D1, D10, D11, D12, D13, D14, D15, D16, D17, D18, D19, D2, D21, D22, D23, D24, D26, D27, D28, D29, D3, D30, D31, D32, D33, D34, D36, D37, D38, D39, D4, D41, D42, D43, D44, D46, D47, D48, D49, D5, D50, D51, D52, D53, D54, D55, D56, D57, D58, D59, D6, D60, D61, D62, D64, D65, D66, D67, D68, D69, D7, D8: moved to B.Cu
- moved R1 325.1 mm to (705.2, 192.5)
- moved U3 323.7 mm to (666.6, 240.9), turned to -90 degrees
- moved C6 323.6 mm to (688.8, 209.2)
- moved C7 323.6 mm to (688.8, 211.8)
- moved C8 315.5 mm to (693.0, 181.4)
- moved C9 315.5 mm to (693.0, 183.9)
- moved C10 313.3 mm to (679.6, 203.2)
- moved C5 312.6 mm to (679.6, 200.6)
- moved C4 312.6 mm to (679.6, 197.9)
- moved C3 312.5 mm to (679.6, 195.3)
- moved C2 312.4 mm to (679.6, 192.6)
- moved C1 312.3 mm to (679.6, 190.0)
- moved J2 306.7 mm to (708.4, 157.1)
- moved C11 302.1 mm to (672.9, 195.7)
- moved C12 302.1 mm to (672.9, 198.2)
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Connections:
- U1 pad 17: /DEBUG -> /DEBUG_RX
- U1 pad 18: /DEBUG -> /DEBUG_TX
Other:
- board outline added: 363.6 x 128.4 mm

Commit message: Verified LCD, power mux, JTAG, USB, and switch matrix
Also changed the switch matrix to use hotswap footprints
Parts:
- removed C18: 1u, Capacitor_SMD:C_0603_1608Metric_Pad1.08x0.95mm_HandSolder
- removed R5: 1M, Resistor_SMD:R_0402_1005Metric
- removed R8: 50, Resistor_SMD:R_0402_1005Metric
- removed TP9: Switch_OUT, TestPoint:TestPoint_Pad_2.5x2.5mm
- added D20: LED, LED_THT:LED_D5.0mm, F.Cu at (704.1, 228.3)
- added D9: LED, LED_THT:LED_D5.0mm, F.Cu at (696.6, 228.3)
- added J3: Conn_01x06_Pin, Connector_PinHeader_2.54mm:PinHeader_1x06_P2.54mm_Vertical, F.Cu at (691.8, 226.9)
- added R10: 1.6k, Resistor_SMD:R_0402_1005Metric, F.Cu at (695.6, 235.1)
- added R11: 100, Resistor_SMD:R_0402_1005Metric, F.Cu at (695.6, 237.1)
- added R9: 1.6k, Resistor_SMD:R_0402_1005Metric, F.Cu at (695.6, 233.1)
- added TP3: Switch_OUT, TestPoint:TestPoint_Pad_2.5x2.5mm, F.Cu at (699.3, 234.4)
- BT1, BT2, BT4: value BA1AAPC -> 1.5V
- C2, C4: value 0.01u -> 0.1u
- D71: footprint LED_SMD:LED_0603_1608Metric_Pad1.05x0.95mm_HandSolder -> LED_THT:LED_D5.0mm
- J2: value Conn_01x05_Pin -> Conn_01x07_Pin
- K1: footprint keebs.pretty-master:Mx_Alps_100 -> MX_Hotswap:MX-Hotswap-1U
- K10: renamed from K46; footprint keebs.pretty-master:Mx_Alps_100 -> MX_Hotswap:MX-Hotswap-1U
- K11: renamed from K51; footprint keebs.pretty-master:Mx_Alps_100 -> MX_Hotswap:MX-Hotswap-1U
- K12: renamed from K56; footprint keebs.pretty-master:Mx_Alps_100 -> MX_Hotswap:MX-Hotswap-1U
- K13: renamed from K61; footprint keebs.pretty-master:Mx_Alps_100 -> MX_Hotswap:MX-Hotswap-1U
- K14: renamed from K66; footprint keebs.pretty-master:Mx_Alps_200 -> MX_Hotswap:MX-Hotswap-2U
- K15: renamed from K2; footprint keebs.pretty-master:Mx_Alps_150 -> MX_Hotswap:MX-Hotswap-1.5U
- K16: renamed from K7; footprint keebs.pretty-master:Mx_Alps_100 -> MX_Hotswap:MX-Hotswap-1U
- K17: renamed from K12; footprint keebs.pretty-master:Mx_Alps_100 -> MX_Hotswap:MX-Hotswap-1U
- K18: renamed from K17; footprint keebs.pretty-master:Mx_Alps_100 -> MX_Hotswap:MX-Hotswap-1U
- K19: renamed from K22; footprint keebs.pretty-master:Mx_Alps_100 -> MX_Hotswap:MX-Hotswap-1U
- K2: renamed from K6; footprint keebs.pretty-master:Mx_Alps_100 -> MX_Hotswap:MX-Hotswap-1U
- K20: renamed from K27; footprint keebs.pretty-master:Mx_Alps_100 -> MX_Hotswap:MX-Hotswap-1U
- K21: renamed from K32; footprint keebs.pretty-master:Mx_Alps_100 -> MX_Hotswap:MX-Hotswap-1U
- K22: renamed from K37; footprint keebs.pretty-master:Mx_Alps_100 -> MX_Hotswap:MX-Hotswap-1U
- K23: renamed from K42; footprint keebs.pretty-master:Mx_Alps_100 -> MX_Hotswap:MX-Hotswap-1U
- K24: renamed from K47; footprint keebs.pretty-master:Mx_Alps_100 -> MX_Hotswap:MX-Hotswap-1U
- K25: renamed from K52; footprint keebs.pretty-master:Mx_Alps_100 -> MX_Hotswap:MX-Hotswap-1U
- K26: renamed from K57; footprint keebs.pretty-master:Mx_Alps_100 -> MX_Hotswap:MX-Hotswap-1U
- K27: renamed from K62; footprint keebs.pretty-master:Mx_Alps_100 -> MX_Hotswap:MX-Hotswap-1U
- K28: renamed from K67; footprint keebs.pretty-master:Mx_Alps_150 -> MX_Hotswap:MX-Hotswap-1.5U
- K29: renamed from K3; footprint keebs.pretty-master:Mx_Alps_175 -> MX_Hotswap:MX-Hotswap-1.75U
- K3: renamed from K11; footprint keebs.pretty-master:Mx_Alps_100 -> MX_Hotswap:MX-Hotswap-1U
- K30: renamed from K8; footprint keebs.pretty-master:Mx_Alps_100 -> MX_Hotswap:MX-Hotswap-1U
- K31: renamed from K13; footprint keebs.pretty-master:Mx_Alps_100 -> MX_Hotswap:MX-Hotswap-1U
- K32: renamed from K18; footprint keebs.pretty-master:Mx_Alps_100 -> MX_Hotswap:MX-Hotswap-1U
- K33: renamed from K23; footprint keebs.pretty-master:Mx_Alps_100 -> MX_Hotswap:MX-Hotswap-1U
- K34: renamed from K28; footprint keebs.pretty-master:Mx_Alps_100 -> MX_Hotswap:MX-Hotswap-1U
- K35: renamed from K33; footprint keebs.pretty-master:Mx_Alps_100 -> MX_Hotswap:MX-Hotswap-1U
- K36: renamed from K38; footprint keebs.pretty-master:Mx_Alps_100 -> MX_Hotswap:MX-Hotswap-1U
- K37: renamed from K43; footprint keebs.pretty-master:Mx_Alps_100 -> MX_Hotswap:MX-Hotswap-1U
- K38: renamed from K48; footprint keebs.pretty-master:Mx_Alps_100 -> MX_Hotswap:MX-Hotswap-1U
- K39: renamed from K53; footprint keebs.pretty-master:Mx_Alps_100 -> MX_Hotswap:MX-Hotswap-1U
- K4: renamed from K16; footprint keebs.pretty-master:Mx_Alps_100 -> MX_Hotswap:MX-Hotswap-1U
- K40: renamed from K58; footprint keebs.pretty-master:Mx_Alps_100 -> MX_Hotswap:MX-Hotswap-1U
- K41: renamed from K68; footprint keebs.pretty-master:Mx_Alps_225 -> MX_Hotswap:MX-Hotswap-2.25U
- K42: renamed from K4; footprint keebs.pretty-master:Mx_Alps_225 -> MX_Hotswap:MX-Hotswap-2.25U
- K43: renamed from K14; footprint keebs.pretty-master:Mx_Alps_100 -> MX_Hotswap:MX-Hotswap-1U
- K44: renamed from K19; footprint keebs.pretty-master:Mx_Alps_100 -> MX_Hotswap:MX-Hotswap-1U
- K45: renamed from K24; footprint keebs.pretty-master:Mx_Alps_100 -> MX_Hotswap:MX-Hotswap-1U
- K46: renamed from K29; footprint keebs.pretty-master:Mx_Alps_100 -> MX_Hotswap:MX-Hotswap-1U
- K47: renamed from K34; footprint keebs.pretty-master:Mx_Alps_100 -> MX_Hotswap:MX-Hotswap-1U
- K48: renamed from K39; footprint keebs.pretty-master:Mx_Alps_100 -> MX_Hotswap:MX-Hotswap-1U
- K49: renamed from K44; footprint keebs.pretty-master:Mx_Alps_100 -> MX_Hotswap:MX-Hotswap-1U
- K5: renamed from K21; footprint keebs.pretty-master:Mx_Alps_100 -> MX_Hotswap:MX-Hotswap-1U
- K50: renamed from K49; footprint keebs.pretty-master:Mx_Alps_100 -> MX_Hotswap:MX-Hotswap-1U
- K51: renamed from K54; footprint keebs.pretty-master:Mx_Alps_100 -> MX_Hotswap:MX-Hotswap-1U
- K52: renamed from K59; footprint keebs.pretty-master:Mx_Alps_100 -> MX_Hotswap:MX-Hotswap-1U
- K53: renamed from K64; footprint keebs.pretty-master:Mx_Alps_150 -> MX_Hotswap:MX-Hotswap-1.5U
- K54: renamed from K69; footprint keebs.pretty-master:Mx_Alps_125 -> MX_Hotswap:MX-Hotswap-1.25U
- K55: renamed from K5; footprint keebs.pretty-master:Mx_Alps_125 -> MX_Hotswap:MX-Hotswap-1.25U
- K56: renamed from K10; footprint keebs.pretty-master:Mx_Alps_125 -> MX_Hotswap:MX-Hotswap-1.25U
- K57: renamed from K15; footprint keebs.pretty-master:Mx_Alps_125 -> MX_Hotswap:MX-Hotswap-1.25U
- K58: renamed from K30; footprint keebs.pretty-master:Mx_Alps_625 -> MX_Hotswap:MX-Hotswap-6.25U
- K59: renamed from K50; footprint keebs.pretty-master:Mx_Alps_125 -> MX_Hotswap:MX-Hotswap-1.25U
- K6: renamed from K26; footprint keebs.pretty-master:Mx_Alps_100 -> MX_Hotswap:MX-Hotswap-1U
- K60: renamed from K55; footprint keebs.pretty-master:Mx_Alps_125 -> MX_Hotswap:MX-Hotswap-1.25U
- K61: renamed from K60; footprint keebs.pretty-master:Mx_Alps_125 -> MX_Hotswap:MX-Hotswap-1.25U
- K62: renamed from K65; footprint keebs.pretty-master:Mx_Alps_125 -> MX_Hotswap:MX-Hotswap-1.25U
- K7: renamed from K31; footprint keebs.pretty-master:Mx_Alps_100 -> MX_Hotswap:MX-Hotswap-1U
- K8: renamed from K36; footprint keebs.pretty-master:Mx_Alps_100 -> MX_Hotswap:MX-Hotswap-1U
- K9: renamed from K41; footprint keebs.pretty-master:Mx_Alps_100 -> MX_Hotswap:MX-Hotswap-1U
- R6: value 330 -> 1.6k
- R7: value 400 -> 750
- SW1: value SW_Push -> SW_RESET
- U1: footprint TM4C123GH6PM:PM0064A_L -> TM4C:QFP50P1200X1200X160-64N
Connections:
- C15 pad 1: /Switch_OUT -> GND
- C15 pad 2: GND -> /Switch_OUT
- D1 pad 1: /row0 -> Net-(D1-K)
- D1 pad 2: Net-(D1-A) -> /row0
- D10 pad 1: /row4 -> Net-(D10-K)
- D10 pad 2: Net-(D10-A) -> /row4
- D11 pad 1: /row0 -> Net-(D11-K)
- D11 pad 2: Net-(D11-A) -> /row0
- D12 pad 1: /row1 -> Net-(D12-K)
- D12 pad 2: Net-(D12-A) -> /row1
- D13 pad 1: /row2 -> Net-(D13-K)
- D13 pad 2: Net-(D13-A) -> /row2
- D14 pad 1: /row3 -> Net-(D14-K)
- D14 pad 2: Net-(D14-A) -> /row3
- D15 pad 1: /row4 -> Net-(D15-K)
- D15 pad 2: Net-(D15-A) -> /row4
- D16 pad 1: /row0 -> Net-(D16-K)
- D16 pad 2: Net-(D16-A) -> /row0
- D17 pad 1: /row1 -> Net-(D17-K)
- D17 pad 2: Net-(D17-A) -> /row1
- D18 pad 1: /row2 -> Net-(D18-K)
- D18 pad 2: Net-(D18-A) -> /row2
- D19 pad 1: /row3 -> Net-(D19-K)
- D19 pad 2: Net-(D19-A) -> /row3
- D2 pad 1: /row1 -> Net-(D2-K)
- D2 pad 2: Net-(D2-A) -> /row1
- D21 pad 1: /row0 -> Net-(D21-K)
- D21 pad 2: Net-(D21-A) -> /row0
- D22 pad 1: /row1 -> Net-(D22-K)
- D22 pad 2: Net-(D22-A) -> /row1
- D23 pad 1: /row2 -> Net-(D23-K)
- D23 pad 2: Net-(D23-A) -> /row2
- D24 pad 1: /row3 -> Net-(D24-K)
- D24 pad 2: Net-(D24-A) -> /row3
- D26 pad 1: /row0 -> Net-(D26-K)
- D26 pad 2: Net-(D26-A) -> /row0
- D27 pad 1: /row1 -> Net-(D27-K)
- D27 pad 2: Net-(D27-A) -> /row1
- D28 pad 1: /row2 -> Net-(D28-K)
- D28 pad 2: Net-(D28-A) -> /row2
- D29 pad 1: /row3 -> Net-(D29-K)
- D29 pad 2: Net-(D29-A) -> /row3
- D3 pad 1: /row2 -> Net-(D3-K)
- D3 pad 2: Net-(D3-A) -> /row2
- D30 pad 1: /row4 -> Net-(D30-K)
- D30 pad 2: Net-(D30-A) -> /row4
- D31 pad 1: /row0 -> Net-(D31-K)
- D31 pad 2: Net-(D31-A) -> /row0
- D32 pad 1: /row1 -> Net-(D32-K)
- D32 pad 2: Net-(D32-A) -> /row1
- D33 pad 1: /row2 -> Net-(D33-K)
- D33 pad 2: Net-(D33-A) -> /row2
- D34 pad 1: /row3 -> Net-(D34-K)
- D34 pad 2: Net-(D34-A) -> /row3
- D36 pad 1: /row0 -> Net-(D36-K)
- D36 pad 2: Net-(D36-A) -> /row0
- D37 pad 1: /row1 -> Net-(D37-K)
- D37 pad 2: Net-(D37-A) -> /row1
- D38 pad 1: /row2 -> Net-(D38-K)
- D38 pad 2: Net-(D38-A) -> /row2
- D39 pad 1: /row3 -> Net-(D39-K)
- D39 pad 2: Net-(D39-A) -> /row3
- D4 pad 1: /row3 -> Net-(D4-K)
- D4 pad 2: Net-(D4-A) -> /row3
- D41 pad 1: /row0 -> Net-(D41-K)
- D41 pad 2: unconnected-(D41-A-Pad2) -> /row0
- D42 pad 1: /row1 -> Net-(D42-K)
- D42 pad 2: Net-(D42-A) -> /row1
- D43 pad 1: /row2 -> Net-(D43-K)
- D43 pad 2: Net-(D43-A) -> /row2
- D44 pad 1: /row3 -> Net-(D44-K)
- D44 pad 2: Net-(D44-A) -> /row3
- D46 pad 1: /row0 -> Net-(D46-K)
- D46 pad 2: Net-(D46-A) -> /row0
- D47 pad 1: /row1 -> Net-(D47-K)
- D47 pad 2: Net-(D47-A) -> /row1
- D48 pad 1: /row2 -> Net-(D48-K)
- D48 pad 2: Net-(D48-A) -> /row2
- D49 pad 1: /row3 -> Net-(D49-K)
- D49 pad 2: Net-(D49-A) -> /row3
- D5 pad 1: /row4 -> Net-(D5-K)
- D5 pad 2: Net-(D5-A) -> /row4
- D50 pad 1: /row4 -> Net-(D50-K)
- D50 pad 2: Net-(D50-A) -> /row4
- D51 pad 1: /row0 -> Net-(D51-K)
- D51 pad 2: Net-(D51-A) -> /row0
- D52 pad 1: /row1 -> Net-(D52-K)
- D52 pad 2: Net-(D52-A) -> /row1
- D53 pad 1: /row2 -> Net-(D53-K)
- D53 pad 2: Net-(D53-A) -> /row2
- D54 pad 1: /row3 -> Net-(D54-K)
- D54 pad 2: Net-(D54-A) -> /row3
- D55 pad 1: /row4 -> Net-(D55-K)
- D55 pad 2: Net-(D55-A) -> /row4
- D56 pad 1: /row0 -> Net-(D56-K)
- D56 pad 2: Net-(D56-A) -> /row0
- D57 pad 1: /row1 -> Net-(D57-K)
- D57 pad 2: Net-(D57-A) -> /row1
- D58 pad 1: /row2 -> Net-(D58-K)
- D58 pad 2: Net-(D58-A) -> /row2
- D59 pad 1: /row3 -> Net-(D59-K)
- D59 pad 2: Net-(D59-A) -> /row3
- D6 pad 1: /row0 -> Net-(D6-K)
- D6 pad 2: Net-(D6-A) -> /row0
- D60 pad 1: /row4 -> Net-(D60-K)
- D60 pad 2: Net-(D60-A) -> /row4
- D61 pad 1: /row0 -> Net-(D61-K)
- D61 pad 2: Net-(D61-A) -> /row0
- D62 pad 1: /row1 -> Net-(D62-K)
- D62 pad 2: Net-(D62-A) -> /row1
- D64 pad 1: /row3 -> Net-(D64-K)
- D64 pad 2: Net-(D64-A) -> /row3
- D65 pad 1: /row4 -> Net-(D65-K)
- D65 pad 2: Net-(D65-A) -> /row4
- D66 pad 1: /row0 -> Net-(D66-K)
- D66 pad 2: Net-(D66-A) -> /row0
- D67 pad 1: /row1 -> Net-(D67-K)
- D67 pad 2: Net-(D67-A) -> /row1
- D68 pad 1: /row2 -> Net-(D68-K)
- D68 pad 2: Net-(D68-A) -> /row2
- D69 pad 1: /row3 -> Net-(D69-K)
- D69 pad 2: Net-(D69-A) -> /row3
- D7 pad 1: /row1 -> Net-(D7-K)
- D7 pad 2: Net-(D7-A) -> /row1
- D8 pad 1: /row2 -> Net-(D8-K)
- D8 pad 2: Net-(D8-A) -> /row2
- IC2 pad 14: /DEBUG_TX -> /BMG220P_DEBUG_TX
- IC2 pad 15: /DEBUG_RX -> /BGM220P_DEBUG_RX
- IC2 pad 3: unconnected-(IC2-PB03-Pad3) -> /~{BLUETOOTH_LED}
- IC2 pad 30: unconnected-(IC2-RESETN-Pad30) -> /BGM220P_RESET
- IC2 pad 4: unconnected-(IC2-PB02-Pad4) -> /BLUETOOTH_TX
- IC2 pad 5: unconnected-(IC2-PB01-Pad5) -> /BLUETOOTH_RX
- J1 pad 4: GND -> unconnected-(J1-ID-Pad4)
- J2 pad 1: GND -> /JTAG_SWCLK_TCLK
- J2 pad 2: /JTAG_SWCLK_TK -> /JTAG_SWDIO_TMS
- J2 pad 3: /JTAG_SWDIO_TMS -> /JTAG_SWO_TDO
- J2 pad 5: /JTAG_SWO_TDO -> /3V3
- K1 pad 2: Net-(D1-A) -> Net-(D1-K)
- K10 pad 2: Net-(D46-A) -> Net-(D46-K)
- K11 pad 2: Net-(D51-A) -> Net-(D51-K)
- K12 pad 2: Net-(D56-A) -> Net-(D56-K)
- K13 pad 2: Net-(D61-A) -> Net-(D61-K)
- K14 pad 2: Net-(D66-A) -> Net-(D66-K)
- K15 pad 2: Net-(D2-A) -> Net-(D2-K)
- K16 pad 2: Net-(D7-A) -> Net-(D7-K)
- K17 pad 2: Net-(D12-A) -> Net-(D12-K)
- K18 pad 2: Net-(D17-A) -> Net-(D17-K)
- K19 pad 2: Net-(D22-A) -> Net-(D22-K)
- K2 pad 2: Net-(D6-A) -> Net-(D6-K)
- K20 pad 2: Net-(D27-A) -> Net-(D27-K)
- K21 pad 2: Net-(D32-A) -> Net-(D32-K)
- K22 pad 2: Net-(D37-A) -> Net-(D37-K)
- K23 pad 2: Net-(D42-A) -> Net-(D42-K)
- K24 pad 2: Net-(D47-A) -> Net-(D47-K)
- K25 pad 2: Net-(D52-A) -> Net-(D52-K)
- K26 pad 2: Net-(D57-A) -> Net-(D57-K)
- K27 pad 2: Net-(D62-A) -> Net-(D62-K)
- K28 pad 2: Net-(D67-A) -> Net-(D67-K)
- K29 pad 2: Net-(D3-A) -> Net-(D3-K)
- K3 pad 2: Net-(D11-A) -> Net-(D11-K)
- K30 pad 2: Net-(D8-A) -> Net-(D8-K)
- K31 pad 2: Net-(D13-A) -> Net-(D13-K)
- K32 pad 2: Net-(D18-A) -> Net-(D18-K)
- K33 pad 2: Net-(D23-A) -> Net-(D23-K)
- K34 pad 2: Net-(D28-A) -> Net-(D28-K)
- K35 pad 2: Net-(D33-A) -> Net-(D33-K)
- K36 pad 2: Net-(D38-A) -> Net-(D38-K)
- K37 pad 2: Net-(D43-A) -> Net-(D43-K)
- K38 pad 2: Net-(D48-A) -> Net-(D48-K)
- K39 pad 2: Net-(D53-A) -> Net-(D53-K)
- K4 pad 2: Net-(D16-A) -> Net-(D16-K)
- K40 pad 2: Net-(D58-A) -> Net-(D58-K)
- K41 pad 2: Net-(D68-A) -> Net-(D68-K)
- K42 pad 2: Net-(D4-A) -> Net-(D4-K)
- K43 pad 2: Net-(D14-A) -> Net-(D14-K)
- K44 pad 2: Net-(D19-A) -> Net-(D19-K)
- K45 pad 2: Net-(D24-A) -> Net-(D24-K)
- K46 pad 2: Net-(D29-A) -> Net-(D29-K)
- K47 pad 2: Net-(D34-A) -> Net-(D34-K)
- K48 pad 2: Net-(D39-A) -> Net-(D39-K)
- K49 pad 2: Net-(D44-A) -> Net-(D44-K)
- K5 pad 2: Net-(D21-A) -> Net-(D21-K)
- K50 pad 2: Net-(D49-A) -> Net-(D49-K)
- K51 pad 2: Net-(D54-A) -> Net-(D54-K)
- K52 pad 2: Net-(D59-A) -> Net-(D59-K)
- K53 pad 2: Net-(D64-A) -> Net-(D64-K)
- K54 pad 2: Net-(D69-A) -> Net-(D69-K)
- K55 pad 2: Net-(D5-A) -> Net-(D5-K)
- K56 pad 2: Net-(D10-A) -> Net-(D10-K)
- K57 pad 2: Net-(D15-A) -> Net-(D15-K)
- K58 pad 2: Net-(D30-A) -> Net-(D30-K)
- K59 pad 2: Net-(D50-A) -> Net-(D50-K)
- K6 pad 2: Net-(D26-A) -> Net-(D26-K)
- K60 pad 2: Net-(D55-A) -> Net-(D55-K)
- K61 pad 2: Net-(D60-A) -> Net-(D60-K)
- K62 pad 2: Net-(D65-A) -> Net-(D65-K)
- K7 pad 2: Net-(D31-A) -> Net-(D31-K)
- K8 pad 2: Net-(D36-A) -> Net-(D36-K)
- K9 pad 2: unconnected-(K41-Pad2) -> Net-(D41-K)
- R1 pad 1: Net-(U1-RST_N) -> /~{RESET}
- SW1 pad 2: Net-(U1-RST_N) -> Net-(R11-Pad2)
- U1 pad 17: /DEBUG_RX -> /TM4C_DEBUG_RX
- U1 pad 18: /DEBUG_TX -> /TM4C_DEBUG_TX
- U1 pad 32: /WAKE -> GND
- U1 pad 34: unconnected-(U1-XOSC0-Pad34) -> GND
- U1 pad 35: unconnected-(U1-GNDX-Pad35) -> GND
- U1 pad 38: Net-(U1-RST_N) -> /~{RESET}
- U1 pad 52: /JTAG_SWCLK_TK -> /JTAG_SWCLK_TCLK
- U1 pad 61: unconnected-(U1-PD0-Pad61) -> /BGM220P_RESET
- U1 pad 62: unconnected-(U1-PD1-Pad62) -> /~{CAPS_LOCK_LED}
- U1 pad 63: unconnected-(U1-PD2-Pad63) -> GND
- U1 pad 64: /SSI_MOSI -> GND

Commit message: Pray to your ECE god of choice
Parts:
- removed BT1, BT2, BT4: 1.5V, BA1AAPC:BAT_BA1AAPC
- removed R11: 100, Resistor_SMD:R_0402_1005Metric
- removed SW1: SW_RESET, Button_Switch_THT:SW_PUSH_6mm
- added J4: Conn_02x05_Odd_Even, Connector_PinHeader_1.27mm:PinHeader_2x05_P1.27mm_Vertical, F.Cu at (691.3, 174.6)
- added J5: BATT_POS, Connector_Pin:Pin_D1.0mm_L10.0mm, B.Cu at (643.3, 177.4)
- added J6: BATT_NEG, Connector_Pin:Pin_D1.0mm_L10.0mm, B.Cu at (643.2, 181.4)
- added SW2: BAT_SWITCH, SLW-121586-5A-D:SLW1215865AD, F.Cu at (690.6, 207.0)
- C6: value 100nF -> 0.1uF
- D1, D10, D11, D12, D13, D14, D15, D16, D17, D18, D19, D2, D21, D22, D23, D24, D26, D27, D28, D29, D3, D30, D31, D32, D33, D34, D36, D37, D38, D39, D4, D41, D42, D43, D44, D46, D47, D48, D49, D5, D50, D51, D52, D53, D54, D55, D56, D57, D58, D59, D6, D60, D61, D62, D64, D65, D66, D67, D68, D69, D7, D8: footprint Diode_SMD:D_0603_1608Metric_Pad1.05x0.95mm_HandSolder -> Diode_SMD:D_SOD-123
- J2: footprint Connector_PinHeader_2.54mm:PinHeader_1x05_P2.54mm_Vertical -> Connector_PinHeader_2.54mm:PinHeader_1x07_P2.54mm_Vertical
- moved TP1 97.6 mm to (659.5, 260.4)
- moved TP2 97.6 mm to (659.5, 265.9)
- moved C17 97.6 mm to (658.2, 254.5)
- moved R3 97.6 mm to (655.1, 254.2)
- moved R4 97.6 mm to (653.1, 254.2)
- moved R7 97.6 mm to (650.6, 256.0)
- moved IC1 96.9 mm to (684.2, 258.3)
- moved C15 96.9 mm to (675.3, 258.2)
- moved C16 96.9 mm to (670.8, 263.7)
- moved C19 96.9 mm to (679.8, 258.2)
- moved D71 96.9 mm to (675.0, 263.7)
- moved R6 96.9 mm to (679.4, 263.7)
- moved TP5 96.9 mm to (670.7, 251.8)
- moved TP6 96.9 mm to (661.1, 251.8)
- moved TP7 96.9 mm to (675.5, 251.8)
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Connections:
- IC2 pad 10: unconnected-(IC2-PA03-Pad10) -> /BGM_SWO
- IC2 pad 26: unconnected-(IC2-PC04-Pad26) -> /PTI_DOUT
- IC2 pad 27: unconnected-(IC2-PC05-Pad27) -> /PTI_DFRAME
- IC2 pad 30: /BGM220P_RESET -> /~{RESET}
- IC2 pad 8: unconnected-(IC2-PA01-Pad8) -> /BGM_SWCLK
- IC2 pad 9: unconnected-(IC2-PA02-Pad9) -> /BGM_SWDIO
- U1 pad 61: /BGM220P_RESET -> GND
Routing:
- net Net-(D41-K): track 0.00 -> 10.4 mm
- added copper zone on F.Cu, net GND
Other:
- board size 363.6 x 128.4 mm -> 335 x 100 mm
- board text added: "All filtering and decoupling is on chip Just connect VDD to 3.3V"
- board text added: "NO COPPER"

Commit message: 6 traces to go :)
Parts:
- J3: moved to B.Cu
- moved TP2 79.0 mm to (654.1, 187.0)
- moved TP1 73.4 mm to (657.9, 187.0)
- moved R4 72.7 mm to (653.7, 181.5)
- moved R3 72.7 mm to (654.9, 181.5)
- moved R10 57.1 mm to (647.7, 176.8), turned to 180 degrees
- moved J5 48.4 mm to (687.3, 197.5), turned to 0 degrees
- moved D20 48.0 mm to (648.4, 181.6)
- moved J3 47.7 mm to (691.9, 196.0)
- moved R7 35.1 mm to (685.7, 254.9), turned to 90 degrees
- moved TP3 32.3 mm to (665.6, 264.3)
- moved D9 31.6 mm to (687.7, 238.8)
- moved R9 29.0 mm to (686.4, 234.8)
- moved C17 22.1 mm to (680.2, 251.9)
- moved R1 16.0 mm to (659.9, 208.0), turned to 180 degrees
- moved D71 16.0 mm to (691.0, 264.5), turned to 180 degrees
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Routing:
- net /row0: track 0.00 -> 482.4 mm, vias 0 -> 1
- net /col0: track 0.00 -> 391.2 mm, vias 0 -> 1
- net /col1: track 0.00 -> 383.6 mm, vias 0 -> 1
- net /row4: track 0.00 -> 354.7 mm, vias 0 -> 1
- net GND: track 0.00 -> 344.2 mm, vias 0 -> 20
- net /row2: track 0.00 -> 339.2 mm, vias 0 -> 13
- net /col2: track 0.00 -> 339.0 mm, vias 0 -> 1
- net /row1: track 0.00 -> 335.6 mm, vias 0 -> 14
- net /row3: track 0.00 -> 330.2 mm, vias 0 -> 10
- net /col3: track 0.00 -> 299.1 mm, vias 0 -> 1
- net /col5: track 0.00 -> 290.0 mm, vias 0 -> 1
- net /col4: track 0.00 -> 277.4 mm, vias 0 -> 1
- net /3V3: track 0.00 -> 270.9 mm, vias 0 -> 14
- net /col6: track 0.00 -> 240.7 mm, vias 0 -> 1
- net /col9: track 0.00 -> 226.5 mm, vias 0 -> 1
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
Commit message: Routed up remaining traces
Parts:
- J4: value Conn_02x05_Odd_Even -> Blue
- moved R9 3.75 mm to (686.4, 231.0)
- moved D62 1.60 mm to (612.2, 206.1)
- moved R10 0.12 mm to (647.6, 176.8)
Routing:
- net /~{CAPS_LOCK_LED}: track 3.91 -> 88.6 mm, vias 1 -> 8
- net /JTAG_TDI: track 20.4 -> 104.6 mm, vias 3 -> 6
- net /JTAG_SWDIO_TMS: track 18.1 -> 100.5 mm, vias 3 -> 6
- net /JTAG_SWCLK_TCLK: track 16.1 -> 98.5 mm, vias 3 -> 6
- net /JTAG_SWO_TDO: track 19.0 -> 98.7 mm, vias 3 -> 6
- net /~{RESET}: track 82.5 -> 131.0 mm, vias 4 -> 9
- net Net-(D9-K): track 4.30 -> 8.05 mm
- net /row2: track 339.2 -> 341.5 mm
- net /col13: track 97.6 -> 99.6 mm, vias 2 -> 1
- net /col7: track 222.2 -> 223.4 mm
- net /col11: track 178.7 -> 179.8 mm
- net Net-(D62-K): track 9.96 -> 9.00 mm
- net /col6: track 240.7 -> 241.7 mm
- net /VBAT: track 76.1 -> 75.2 mm
- net /row1: track 335.6 -> 334.7 mm
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