File: hw/KeyboardPCB/KeyboardPCB.kicad_pcb (KiCad board)
At the start: 2 copper layers, 335 x 100 mm, 173 parts, among them IC1 TPS2113ADRBR, IC2 BGM220PC22HNA2R, J1 USB_B_Micro, J2 Conn_01x07_Pin, J3 Conn_01x06_Pin, J4 Blue, J5 BATT_POS, J6 BATT_NEG, K1 KEYSW, K10 KEYSW, K11 KEYSW, K12 KEYSW, K13 KEYSW, K14 KEYSW, K15 KEYSW, K16 KEYSW, K17 KEYSW, K18 KEYSW, K19 KEYSW, K2 KEYSW, K20 KEYSW, K21 KEYSW, K22 KEYSW, K23 KEYSW, K24 KEYSW, K25 KEYSW, K26 KEYSW, K27 KEYSW, K28 KEYSW, K29 KEYSW, K3 KEYSW, K30 KEYSW, K31 KEYSW, K32 KEYSW, K33 KEYSW, K34 KEYSW, K35 KEYSW, K36 KEYSW, K37 KEYSW, K38 KEYSW, K39 KEYSW, K4 KEYSW, K40 KEYSW, K41 KEYSW, K42 KEYSW, K43 KEYSW, K44 KEYSW, K45 KEYSW, K46 KEYSW, K47 KEYSW, K48 KEYSW, K49 KEYSW, K5 KEYSW, K50 KEYSW, K51 KEYSW, K52 KEYSW, K53 KEYSW, K54 KEYSW, K55 KEYSW, K56 KEYSW, K57 KEYSW, K58 KEYSW, K59 KEYSW, K6 KEYSW, K60 KEYSW, K61 KEYSW, K62 KEYSW, K7 KEYSW, K8 KEYSW, K9 KEYSW, SW2 BAT_SWITCH, U1 TM4C123GH6PMI7, U2 TPS73633DBV, U3 Adafruit ST7735R, X2 16MHz

Commit message: Added EM4_WAKEUP signal from PD0 (TM4C) to PC0 (BGM)
Parts:
- J4: value Blue -> Conn_02x05_Odd_Even
Connections:
- IC2 pad 22: unconnected-(IC2-PC00-Pad22) -> /EM4_WAKEUP
- U1 pad 61: GND -> /EM4_WAKEUP
Routing:
- net /EM4_WAKEUP: track 0.00 -> 75.4 mm, vias 0 -> 4
- net GND: track 344.2 -> 342.3 mm
Changed lines of the file:
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@@
   (net 115 "unconnected-(IC2-PD02-Pad19)")
   (net 116 "unconnected-(IC2-NC-Pad21)")
-  (net 117 "unconnected-(IC2-PC00-Pad22)")
+  (net 117 "/EM4_WAKEUP")
   (net 118 "unconnected-(IC2-PC01-Pad23)")
   (net 119 "unconnected-(IC2-PC02-Pad24)")
@@
       (net 101 "/col9") (pinfunction "PE5") (pintype "bidirectional"))
     (pad "61" smd rect (at -2.25 -5.738) (size 0.3 1.475) (layers "F.Cu" "F.Paste" "F.Mask")
-      (net 1 "GND") (pinfunction "PD0") (pintype "bidirectional"))
+      (net 117 "/EM4_WAKEUP") (pinfunction "PD0") (pintype "bidirectional"))
     (pad "62" smd rect (at -2.75 -5.738) (size 0.3 1.475) (layers "F.Cu" "F.Paste" "F.Mask")
       (net 145 "/~{CAPS_LOCK_LED}") (pinfunction "PD1") (pintype "bidirectional"))
@@
         (effects (font (size 0.8 0.5) (thickness 0.125)))
     )
-    (fp_text value "Blue" (at 0.635 6.775) (layer "F.Fab")
+    (fp_text value "Conn_02x05_Odd_Even" (at 0.635 6.775) (layer "F.Fab")
         (effects (font (size 0.5 0.5) (thickness 0.125)))
     )
@@
       (net 116 "unconnected-(IC2-NC-Pad21)") (pinfunction "NC") (pintype "no_connect"))
     (pad "22" smd oval (at 5.65 4.1 90) (size 0.8 2.4) (layers "F.Cu" "F.Paste" "F.Mask")
-      (net 117 "unconnected-(IC2-PC00-Pad22)") (pinfunction "PC00") (pintype "passive+no_connect"))
+      (net 117 "/EM4_WAKEUP") (pinfunction "PC00") (pintype "passive"))
     (pad "23" smd oval (at 5.65 2.9 90) (size 0.8 2.4) (layers "F.Cu" "F.Paste" "F.Mask")
       (net 118 "unconnected-(IC2-PC01-Pad23)") (pinfunction "PC01") (pintype "passive+no_connect"))
@@
   (segment (start 673.698 195.6805) (end 673.7375 195.72) (width 0.254) (layer "F.Cu") (net 1))
   (segment (start 679.098 197.779) (end 679.098 200.433) (width 0.254) (layer "F.Cu") (net 1))
-  (segment (start 652.123 195.829) (end 652.123 193.941) (width 0.254) (layer "F.Cu") (net 1))
   (segment (start 679.098 200.433) (end 679.098 203.087) (width 0.254) (layer "F.Cu") (net 1))
   (segment (start 663.2855 198.2165) (end 663.323 198.254) (width 0.254) (layer "F.Cu") (net 1))
@@
   (segment (start 662.1369 182.0651) (end 662.323 181.879) (width 0.1778) (layer "B.Cu") (net 108))
   (segment (start 689.073 181.129) (end 681.4485 188.7535) (width 0.1778) (layer "B.Cu") (net 108))
+  (segment (start 687.442293 181.998293) (end 685.269907 181.998293) (width 0.1778) (layer "F.Cu") (net 109))
+  (segment (start 685.269907 181.998293) (end 677.448 189.8202) (width 0.1778) (layer "F.Cu") (net 109))
   (segment (start 664.373 183.079) (end 662.548748 183.079) (width 0.1778) (layer "F.Cu") (net 109))
-  (segment (start 685.7642 181.504) (end 687.448 181.504) (width 0.1778) (layer "F.Cu") (net 109))
-  (segment (start 677.448 189.8202) (end 685.7642 181.504) (width 0.1778) (layer "F.Cu") (net 109))
   (segment (start 661.598748 182.129) (end 660.698 182.129) (width 0.1778) (layer "F.Cu") (net 109))
   (segment (start 662.548748 183.079) (end 661.598748 182.129) (width 0.1778) (layer "F.Cu") (net 109))
   (via (at 677.448 189.8202) (size 0.5) (drill 0.3) (layers "F.Cu" "B.Cu") (net 109))
-  (via (at 687.448 181.504) (size 0.5) (drill 0.3) (layers "F.Cu" "B.Cu") (net 109))
+  (via (at 687.442293 181.998293) (size 0.5) (drill 0.3) (layers "F.Cu" "B.Cu") (net 109))
   (via (at 660.698 182.129) (size 0.5) (drill 0.3) (layers "F.Cu" "B.Cu") (net 109))
-  (segment (start 690.543 178.409) (end 691.303 178.409) (width 0.1778) (layer "B.Cu") (net 109))
+  (segment (start 687.442293 181.998293) (end 687.442293 181.509707) (width 0.1778) (layer "B.Cu") (net 109))
   (segment (start 677.3892 189.879) (end 677.448 189.8202) (width 0.1778) (layer "B.Cu") (net 109))
   (segment (start 660.698 188.629) (end 661.948 189.879) (width 0.1778) (layer "B.Cu") (net 109))
+  (segment (start 687.442293 181.509707) (end 690.543 178.409) (width 0.1778) (layer "B.Cu") (net 109))
   (segment (start 660.698 182.129) (end 660.698 188.629) (width 0.1778) (layer "B.Cu") (net 109))
-  (segment (start 687.448 181.504) (end 690.543 178.409) (width 0.1778) (layer "B.Cu") (net 109))
+  (segment (start 690.543 178.409) (end 691.303 178.409) (width 0.1778) (layer "B.Cu") (net 109))
   (segment (start 661.948 189.879) (end 677.3892 189.879) (width 0.1778) (layer "B.Cu") (net 109))
   (segment (start 662.348 184.279) (end 661.448 183.379) (width 0.1778) (layer "F.Cu") (net 110))
@@
   (segment (start 661.448 183.379) (end 661.0758 183.7512) (width 0.1778) (layer "B.Cu") (net 110))
   (segment (start 661.0758 188.3818) (end 662.0758 189.3818) (width 0.1778) (layer "B.Cu") (net 110))
+  (segment (start 660.9869 206.2151) (end 666.0147 206.2151) (width 0.1778) (layer "F.Cu") (net 117))
+  (segment (start 660.323 206.879) (end 660.9869 206.2151) (width 0.1778) (layer "F.Cu") (net 117))
+  (segment (start 688.778393 181.459393) (end 685.242607 181.459393) (width 0.1778) (layer "F.Cu") (net 117))
+  (segment (start 652.123 195.16688) (end 653.948 196.99188) (width 0.1778) (layer "F.Cu") (net 117))
+  (segment (start 652.123 193.941) (end 652.123 195.16688) (width 0.1778) (layer "F.Cu") (net 117))
+  (segment (start 666.0147 206.2151) (end 670.323 201.9068) (width 0.1778) (layer "F.Cu") (net 117))
+  (segment (start 689.448 182.129) (end 688.778393 181.459393) (width 0.1778) (layer "F.Cu") (net 117))
+  (segment (start 685.242607 181.459393) (end 682.423 184.279) (width 0.1778) (layer "F.Cu") (net 117))
+  (segment (start 653.948 196.99188) (end 653.948 202.5424) (width 0.1778) (layer "F.Cu") (net 117))
+  (segment (start 670.323 201.9068) (end 670.323 197.129) (width 0.1778) (layer "F.Cu") (net 117))
+  (segment (start 682.423 184.279) (end 675.673 184.279) (width 0.1778) (layer "F.Cu") (net 117))
+  (via (at 670.323 197.129) (size 0.5) (drill 0.3) (layers "F.Cu" "B.Cu") (net 117))
+  (via (at 689.448 182.129) (size 0.5) (drill 0.3) (layers "F.Cu" "B.Cu") (net 117))
+  (via (at 653.948 202.5424) (size 0.5) (drill 0.3) (layers "F.Cu" "B.Cu") (net 117))
+  (via (at 660.323 206.879) (size 0.5) (drill 0.3) (layers "F.Cu" "B.Cu") (net 117))
+  (segment (start 680.39698 190.6679) (end 680.9091 190.6679) (width 0.1778) (layer "B.Cu") (net 117))
+  (segment (start 656.87352 202.5424) (end 660.323 205.99188) (width 0.1778) (layer "B.Cu") (net 117))
+  (segment (start 680.9091 190.6679) (end 689.448 182.129) (width 0.1778) (layer "B.Cu") (net 117))
+  (segment (start 660.323 205.99188) (end 660.323 206.879) (width 0.1778) (layer "B.Cu") (net 117))
+  (segment (start 670.323 197.129) (end 673.93588 197.129) (width 0.1778) (layer "B.Cu") (net 117))
+  (segment (start 653.948 202.5424) (end 656.87352 202.5424) (width 0.1778) (layer "B.Cu") (net 117))
+  (segment (start 673.93588 197.129) (end 680.39698 190.6679) (width 0.1778) (layer "B.Cu") (net 117))
   (segment (start 692.573 179.679) (end 691.623 180.629) (width 0.1778) (layer "F.Cu") (net 121))
   (segment (start 683.923 179.479) (end 675.673 179.479) (width 0.1778) (layer "F.Cu") (net 121))
