File: hw/KeyboardPCB/KeyboardPCB.kicad_sch (KiCad schematic)
At the start: 173 parts, among them J1 USB_B_Micro, J2 Conn_01x05_Pin, K1 KEYSW, K10 KEYSW, K11 KEYSW, K12 KEYSW, K13 KEYSW, K14 KEYSW, K15 KEYSW, K16 KEYSW, K17 KEYSW, K18 KEYSW, K19 KEYSW, K2 KEYSW, K20 KEYSW, K21 KEYSW, K22 KEYSW, K23 KEYSW, K24 KEYSW, K25 KEYSW, K26 KEYSW, K27 KEYSW, K28 KEYSW, K29 KEYSW, K3 KEYSW, K30 KEYSW, K31 KEYSW, K32 KEYSW, K33 KEYSW, K34 KEYSW, K35 KEYSW, K36 KEYSW, K37 KEYSW, K38 KEYSW, K39 KEYSW, K4 KEYSW, K40 KEYSW, K41 KEYSW, K42 KEYSW, K43 KEYSW, K44 KEYSW, K45 KEYSW, K46 KEYSW, K47 KEYSW, K48 KEYSW, K49 KEYSW, K5 KEYSW, K50 KEYSW, K51 KEYSW, K52 KEYSW, K53 KEYSW, K54 KEYSW, K55 KEYSW, K56 KEYSW, K57 KEYSW, K58 KEYSW, K59 KEYSW, K6 KEYSW, K60 KEYSW, K61 KEYSW, K62 KEYSW, K63 KEYSW, K64 KEYSW, K65 KEYSW, K66 KEYSW, K67 KEYSW, K68 KEYSW, K69 KEYSW, K7 KEYSW, K70 KEYSW, K8 KEYSW, K9 KEYSW, SW1 SW_Push, U1 TM4C123GH6PMI7, U2 TPS73633DBV, U3 Adafruit ST7735R, X2 16MHz

Commit message: PCB update
Parts:
- added BT1, BT2, BT4: BA1AAPC, BA1AAPC:BAT_BA1AAPC, symbol BA1AAPC:BA1AAPC
- added C17, C19: 0.1u, Capacitor_SMD:C_0603_1608Metric_Pad1.08x0.95mm_HandSolder, symbol Device:C
- added C18: 1u, Capacitor_SMD:C_0603_1608Metric_Pad1.08x0.95mm_HandSolder, symbol Device:C
- added IC1: TPS2113ADRBR, SON65P300X300X100-9N-D, symbol TPS2113ADRBR:TPS2113ADRBR
- added R5: 1M, Resistor_SMD:R_0402_1005Metric, symbol Device:R
- added R7: 400, Resistor_SMD:R_0402_1005Metric, symbol Device:R
- added R8: 50, Resistor_SMD:R_0402_1005Metric, symbol Device:R
- C1, C10, C11, C12, C13, C14, C2, C3, C4, C5, C8, C9: footprint (none) -> Capacitor_SMD:C_0603_1608Metric_Pad1.08x0.95mm_HandSolder
- C6, C7: footprint Capacitor_SMD:C_0402_1005Metric -> Capacitor_SMD:C_0603_1608Metric_Pad1.08x0.95mm_HandSolder
- D1, D10, D11, D12, D13, D14, D15, D16, D17, D18, D19, D2, D20, D21, D22, D23, D24, D25, D26, D27, D28, D29, D3, D30, D31, D32, D33, D34, D35, D36, D37, D38, D39, D4, D40, D41, D42, D43, D44, D45, D46, D47, D48, D49, D5, D50, D51, D52, D53, D54, D55, D56, D57, D58, D59, D6, D60, D61, D62, D63, D64, D65, D66, D67, D68, D69, D7, D70, D8, D9: footprint (none) -> Diode_SMD:D_0603_1608Metric_Pad1.05x0.95mm_HandSolder
- J1: footprint (none) -> Connector_USB:USB_Micro-B_Amphenol_10103594-0001LF_Horizontal
- K1: footprint (none) -> keebs.pretty-master:Mx_Alps_100
Connections:
- net 3V3: now also R5.2
- net GND: now also BT2.-, C17.2, C18.2, C19.2, IC1.2 (~{EN}), IC1.3 (VSNS), IC1.5 (GND_1), IC1.9 (GND_2), R7.2, R8.2
- net VBUS: now also C17.1, IC1.8 (IN1); no longer C15.1, TP3.1, TP4.1, U2.1 (IN), U2.3 (EN)
- net WAKE: now reaches U1.32 (WAKE_N)
- net WAKE: now also R5.1
- new net: BT1.+, BT4.-
- new net: IC1.4 (ILIM), R7.1
- new net: BT1.-, BT2.+
- new net Switch_OUT: C15.1, C18.1, IC1.7 (OUT), R8.1, TP3.1, TP4.1, U2.1 (IN), U2.3 (EN)
- new net VBAT: BT4.+, C19.1, IC1.6 (IN2)
- no-connect marks 0 -> 1
Other:
- moved on the sheet: J2

Commit message: Added remaining footprints and aligned keys on layout
Parts:
- removed D20, D25, D35, D40, D45, D63, D70, D9: D, Diode_SMD:D_0603_1608Metric_Pad1.05x0.95mm_HandSolder, symbol Device:D
- removed K20, K25, K35, K40, K45, K63, K70, K9: KEYSW, symbol keyboard_parts:KEYSW
- added IC2: BGM220PC22HNA2R, BGM220PC22HNA2R, symbol BGM220PC22HNA2R:BGM220PC22HNA2R
- added TP5: 3V3, TestPoint:TestPoint_Pad_2.5x2.5mm, symbol Connector:TestPoint
- added TP6: GND, TestPoint:TestPoint_Pad_2.5x2.5mm, symbol Connector:TestPoint
- added TP7: IN1, TestPoint:TestPoint_Pad_2.5x2.5mm, symbol Connector:TestPoint
- added TP8: VBAT, TestPoint:TestPoint_Pad_2.5x2.5mm, symbol Connector:TestPoint
- added TP9: Switch_OUT, TestPoint:TestPoint_Pad_2.5x2.5mm, symbol Connector:TestPoint
- D71: footprint (none) -> LED_SMD:LED_0603_1608Metric_Pad1.05x0.95mm_HandSolder
- IC1: footprint SON65P300X300X100-9N-D -> SwitchingICLibrary:SON65P300X300X100-9N-D
- K10, K15, K5, K50, K55, K60, K65, K69: footprint (none) -> keebs.pretty-master:Mx_Alps_125
- K11, K12, K13, K14, K16, K17, K18, K19, K21, K22, K23, K24, K26, K27, K28, K29, K31, K32, K33, K34, K36, K37, K38, K39, K41, K42, K43, K44, K46, K47, K48, K49, K51, K52, K53, K54, K56, K57, K58, K59, K6, K61, K62, K7, K8: footprint (none) -> keebs.pretty-master:Mx_Alps_100
- K2, K64, K67: footprint (none) -> keebs.pretty-master:Mx_Alps_150
- K3: footprint (none) -> keebs.pretty-master:Mx_Alps_175
- K30: footprint (none) -> keebs.pretty-master:Mx_Alps_625
- K4, K68: footprint (none) -> keebs.pretty-master:Mx_Alps_225
- K66: footprint (none) -> keebs.pretty-master:Mx_Alps_200
- SW1: footprint (none) -> Button_Switch_THT:SW_PUSH_6mm
- TP1, TP2, TP3, TP4: footprint (none) -> TestPoint:TestPoint_Pad_2.5x2.5mm
- X2: footprint (none) -> CrystalLibrary:NX5032GA16000000MHZLNCD1
Connections:
- net 3V3: now also TP5.1
- net GND: now also TP6.1
- net Switch_OUT: now also TP9.1
- net VBAT: now also TP8.1
- net VBUS: now also TP7.1
Other:
- moved on the sheet: K30

Commit message: Made outline and placed all components in position. Just need to route :)
Parts:
- removed TP3: EN, TestPoint:TestPoint_Pad_2.5x2.5mm, symbol Connector:TestPoint
- removed TP4: VBUS, TestPoint:TestPoint_Pad_2.5x2.5mm, symbol Connector:TestPoint
- IC2: footprint BGM220PC22HNA2R -> BluetoothModuleLibrary:BGM220PC22HNA2R
Connections:
- net 3V3: now also IC2.13 (VDD)
- net GND: now also IC2.1 (GND_1), IC2.12 (GND_2), IC2.20 (GND_3), IC2.31 (GND_4)
- net DEBUG_TX: now reaches IC2.14 (PA05)
- net DEBUG_TX: now also U1.18 (PA1_U0Tx)
- net DEBUG_RX: now reaches IC2.15 (PA06)
- net DEBUG_RX: now also U1.17 (PA0_U0Rx)
- removed net DEBUG: U1.17 (PA0_U0Rx), U1.18 (PA1_U0Tx)
Changed lines of the file:
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@@
   (junction (at 560.07 121.92) (diameter 0) (color 0 0 0 0)
   )
-  (junction (at 45.72 43.18) (diameter 0) (color 0 0 0 0)
-  )
   (junction (at 494.03 139.7) (diameter 0) (color 0 0 0 0)
   )
@@
     (stroke (width 0) (type default))
   )
-  (wire (pts (xy 45.72 43.18) (xy 39.37 43.18))
-    (stroke (width 0) (type default))
-  )
   (wire (pts (xy 494.03 80.01) (xy 494.03 85.09))
     (stroke (width 0) (type default))
@@
     (stroke (width 0) (type default))
   )
+  (wire (pts (xy 281.94 261.62) (xy 288.29 261.62))
+    (stroke (width 0) (type default))
+  )
   (wire (pts (xy 386.08 85.09) (xy 386.08 102.87))
     (stroke (width 0) (type default))
@@
     (stroke (width 0) (type default))
   )
-  (wire (pts (xy 54.61 43.18) (xy 45.72 43.18))
+  (wire (pts (xy 39.37 43.18) (xy 54.61 43.18))
     (stroke (width 0) (type default))
   )
@@
     (stroke (width 0) (type default))
   )
+  (wire (pts (xy 281.94 260.35) (xy 281.94 261.62))
+    (stroke (width 0) (type default))
+  )
   (wire (pts (xy 158.75 256.54) (xy 162.56 256.54))
     (stroke (width 0) (type default))
@@
     (effects (font (size 3 3) (thickness 0.254) bold (color 0 4 255 1)) (justify top))
   )
+  (label "DEBUG_RX" (at 288.29 269.24 180) (fields_autoplaced)
+    (effects (font (size 1.27 1.27)) (justify right bottom))
+  )
   (label "col9" (at 472.44 80.01 0) (fields_autoplaced)
     (effects (font (size 1.27 1.27)) (justify left bottom))
@@
     (effects (font (size 1.27 1.27)) (justify right bottom))
   )
-  (label "DEBUG" (at 116.84 139.7 180) (fields_autoplaced)
+  (label "DEBUG_TX" (at 116.84 139.7 180) (fields_autoplaced)
     (effects (font (size 1.27 1.27)) (justify right bottom))
   )
@@
     (effects (font (size 1.27 1.27)) (justify left bottom))
   )
-  (label "DEBUG" (at 116.84 137.16 180) (fields_autoplaced)
+  (label "DEBUG_RX" (at 116.84 137.16 180) (fields_autoplaced)
     (effects (font (size 1.27 1.27)) (justify right bottom))
   )
@@
     (effects (font (size 1.27 1.27) bold) (justify right bottom))
   )
+  (label "DEBUG_TX" (at 288.29 266.7 180) (fields_autoplaced)
+    (effects (font (size 1.27 1.27)) (justify right bottom))
+  )
   (label "col7" (at 429.26 80.01 0) (fields_autoplaced)
     (effects (font (size 1.27 1.27)) (justify left bottom))
@@
     (effects (font (size 1.27 1.27)) (justify right bottom))
   )
+  (label "3V3" (at 288.29 264.16 180) (fields_autoplaced)
+    (effects (font (size 1.27 1.27) bold) (justify right bottom))
+  )
   (label "col2" (at 116.84 177.8 180) (fields_autoplaced)
     (effects (font (size 1.27 1.27)) (justify right bottom))
@@
     )
   )
-  (symbol (lib_id "Connector:TestPoint") (at 39.37 43.18 0) (unit 1)
-    (in_bom yes) (on_board yes) (dnp no)
-    (property "Reference" "TP3" (at 38.1 38.1 0)
-      (effects (font (size 1.27 1.27)) (justify left))
-    )
-    (property "Value" "EN" (at 35.56 40.64 0)
-      (effects (font (size 1.27 1.27)) (justify left))
-    )
-    (property "Footprint" "TestPoint:TestPoint_Pad_2.5x2.5mm" (at 44.45 43.18 0)
-      (effects (font (size 1.27 1.27)) hide)
-    )
-    (property "Datasheet" "~" (at 44.45 43.18 0)
-      (effects (font (size 1.27 1.27)) hide)
-    )
-    (pin "1")
-    (instances
-      (project "KeyboardPCB"
-        (path "/2d193c8d-36cd-4337-adc1-05f8d95a4b88"
-          (reference "TP3") (unit 1)
-        )
-      )
-    )
-  )
   (symbol (lib_id "power:GND") (at 173.99 238.76 0) (unit 1)
     (in_bom yes) (on_board yes) (dnp no) (fields_autoplaced)
@@
     )
   )
+  (symbol (lib_id "power:GND") (at 321.31 269.24 90) (unit 1)
+    (in_bom yes) (on_board yes) (dnp no) (fields_autoplaced)
+    (property "Reference" "#PWR025" (at 327.66 269.24 0)
+      (effects (font (size 1.27 1.27)) hide)
+    )
+    (property "Value" "GND" (at 325.12 269.24 90)
+      (effects (font (size 1.27 1.27)) (justify right))
+    )
+    (property "Footprint" "" (at 321.31 269.24 0)
+      (effects (font (size 1.27 1.27)) hide)
+    )
+    (property "Datasheet" "" (at 321.31 269.24 0)
+      (effects (font (size 1.27 1.27)) hide)
+    )
+    (pin "1")
+    (instances
+      (project "KeyboardPCB"
+        (path "/2d193c8d-36cd-4337-adc1-05f8d95a4b88"
+          (reference "#PWR025") (unit 1)
+        )
+      )
+    )
+  )
   (symbol (lib_id "keyboard_parts:KEYSW") (at 443.23 85.09 0) (unit 1)
     (in_bom yes) (on_board yes) (dnp no) (fields_autoplaced)
@@
     )
   )
-  (symbol (lib_id "Connector:TestPoint") (at 45.72 43.18 0) (unit 1)
-    (in_bom yes) (on_board yes) (dnp no)
-    (property "Reference" "TP4" (at 44.45 38.1 0)
-      (effects (font (size 1.27 1.27)) (justify left))
-    )
-    (property "Value" "VBUS" (at 46.99 41.91 0)
-      (effects (font (size 1.27 1.27)) (justify left))
-    )
-    (property "Footprint" "TestPoint:TestPoint_Pad_2.5x2.5mm" (at 50.8 43.18 0)
-      (effects (font (size 1.27 1.27)) hide)
-    )
-    (property "Datasheet" "~" (at 50.8 43.18 0)
-      (effects (font (size 1.27 1.27)) hide)
-    )
-    (pin "1")
-    (instances
-      (project "KeyboardPCB"
-        (path "/2d193c8d-36cd-4337-adc1-05f8d95a4b88"
-          (reference "TP4") (unit 1)
-        )
-      )
-    )
-  )
   (symbol (lib_id "keyboard_parts:KEYSW") (at 266.7 157.48 0) (unit 1)
     (in_bom yes) (on_board yes) (dnp no) (fields_autoplaced)
@@
     )
   )
+  (symbol (lib_id "power:GND") (at 288.29 233.68 270) (unit 1)
+    (in_bom yes) (on_board yes) (dnp no) (fields_autoplaced)
+    (property "Reference" "#PWR023" (at 281.94 233.68 0)
+      (effects (font (size 1.27 1.27)) hide)
+    )
+    (property "Value" "GND" (at 284.48 233.68 90)
+      (effects (font (size 1.27 1.27)) (justify right))
+    )
+    (property "Footprint" "" (at 288.29 233.68 0)
+      (effects (font (size 1.27 1.27)) hide)
+    )
+    (property "Datasheet" "" (at 288.29 233.68 0)
+      (effects (font (size 1.27 1.27)) hide)
+    )
+    (pin "1")
+    (instances
+      (project "KeyboardPCB"
+        (path "/2d193c8d-36cd-4337-adc1-05f8d95a4b88"
+          (reference "#PWR023") (unit 1)
+        )
+      )
+    )
+  )
   (symbol (lib_id "BGM220PC22HNA2R:BGM220PC22HNA2R") (at 288.29 233.68 0) (unit 1)
     (in_bom yes) (on_board yes) (dnp no) (fields_autoplaced)
@@
       (effects (font (size 1.27 1.27)))
     )
-    (property "Footprint" "BGM220PC22HNA2R" (at 317.5 328.6 0)
+    (property "Footprint" "BluetoothModuleLibrary:BGM220PC22HNA2R" (at 317.5 328.6 0)
       (effects (font (size 1.27 1.27)) (justify left top) hide)
     )
@@
     )
   )
+  (symbol (lib_id "power:GND") (at 321.31 241.3 90) (unit 1)
+    (in_bom yes) (on_board yes) (dnp no) (fields_autoplaced)
+    (property "Reference" "#PWR024" (at 327.66 241.3 0)
+      (effects (font (size 1.27 1.27)) hide)
+    )
+    (property "Value" "GND" (at 325.12 241.3 90)
+      (effects (font (size 1.27 1.27)) (justify right))
+    )
+    (property "Footprint" "" (at 321.31 241.3 0)
+      (effects (font (size 1.27 1.27)) hide)
+    )
+    (property "Datasheet" "" (at 321.31 241.3 0)
+      (effects (font (size 1.27 1.27)) hide)
+    )
+    (pin "1")
+    (instances
+      (project "KeyboardPCB"
+        (path "/2d193c8d-36cd-4337-adc1-05f8d95a4b88"
+          (reference "#PWR024") (unit 1)
+        )
+      )
+    )
+  )
   (symbol (lib_id "keyboard_parts:KEYSW") (at 508 85.09 0) (unit 1)
     (in_bom yes) (on_board yes) (dnp no) (fields_autoplaced)
@@
         )
       )
+    )
+  )
+  (symbol (lib_id "power:GND") (at 281.94 260.35 270) (unit 1)
+    (in_bom yes) (on_board yes) (dnp no) (fields_autoplaced)
+    (property "Reference" "#PWR026" (at 275.59 260.35 0)
+      (effects (font (size 1.27 1.27)) hide)
+    )
+    (property "Value" "GND" (at 278.13 260.35 90)
+      (effects (font (size 1.27 1.27)) (justify right))
+    )
+    (property "Footprint" "" (at 281.94 260.35 0)
+      (effects (font (size 1.27 1.27)) hide)
+    )
+    (property "Datasheet" "" (at 281.94 260.35 0)
+      (effects (font (size 1.27 1.27)) hide)
+    )
+    (pin "1")
+    (instances
+      (project "KeyboardPCB"
+        (path "/2d193c8d-36cd-4337-adc1-05f8d95a4b88"
+          (reference "#PWR026") (unit 1)
+        )
+      )

Commit message: Verified regulator circuit, added LEDs based on BOM
Parts:
- added D20, D9: LED, LED_THT:LED_D5.0mm, symbol Device:LED
- added J3: Conn_01x06_Pin, Connector_PinHeader_2.54mm:PinHeader_1x06_P2.54mm_Vertical, symbol Connector:Conn_01x06_Pin
- added R10, R9: 1.6k, Resistor_SMD:R_0402_1005Metric, symbol Device:R
- BT1, BT2, BT4: value BA1AAPC -> 1.5V
- D71: footprint LED_SMD:LED_0603_1608Metric_Pad1.05x0.95mm_HandSolder -> LED_THT:LED_D5.0mm; If (none) -> 1mA; Part (none) -> HLMP-D150; Vf (none) -> 1.7V
- R6: value 330 -> 1.6k
Connections:
- net 3V3: now also D20.2 (A), D9.2 (A)
- net BLUETOOTH_RX: now also IC2.5 (PB01), J3.5 (Pin_5)
- net BLUETOOTH_TX: now also IC2.4 (PB02), J3.6 (Pin_6)
- net GND: now also C15.1; no longer C15.2
- net Switch_OUT: now also C15.2; no longer C15.1
- net at K41.2: now also D41.2 (A)
- net ~{BLUETOOTH_LED}: now reaches IC2.3 (PB03)
- net ~{BLUETOOTH_LED}: now also R10.1
- net BGM220P_RESET: now reaches IC2.30 (RESETN)
- net BGM220P_RESET: now also U1.61 (PD0)
- net ~{CAPS_LOCK_LED}: now reaches U1.62 (PD1)
- net ~{CAPS_LOCK_LED}: now also R9.1
- net AIN5: now reaches U1.63 (PD2)
- net DEBUG_RX renamed BGM220P_DEBUG_RX
- net BGM220P_DEBUG_RX: now also J3.1 (Pin_1); no longer U1.17 (PA0_U0Rx)
- net DEBUG_TX renamed BMG220P_DEBUG_TX
- net BMG220P_DEBUG_TX: now also J3.2 (Pin_2); no longer U1.18 (PA1_U0Tx)
- net SSI_MOSI: no longer names the net of U1.64 (PD3)
- new net: D9.1 (K), R9.2
- new net: D20.1 (K), R10.2
- new net TM4C_DEBUG_RX: J3.3 (Pin_3), U1.17 (PA0_U0Rx)
- new net TM4C_DEBUG_TX: J3.4 (Pin_4), U1.18 (PA1_U0Tx)
- no-connect marks 1 -> 26
Other:
- note added: "PB2 is BGM220P RX PB1 is BGM220P TX BLUETOOTH_?X is relative to the TM4C"
- moved on the sheet: C15, IC2, J2
